File: LaserPointer.kicad_sch (KiCad schematic)
At the start: 10 parts, among them J1 Laser Diode - 5mW 650nm Red, SW1 Mini Soft Touch Push-button S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, U1 MCP1640Bx-xCHY

Commit message: Made board WAY smaller to be chcheaper, uses battery terminals now lol. Just solder leads on and use a holder
Parts:
- BT1: footprint Mylibrary:BatteryHolder_Keystone_1020_1xAAA -> Mylibrary:Batt terminal pads
Changed lines of the file:
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@@
 			)
 		)
-		(property "Footprint" "Mylibrary:BatteryHolder_Keystone_1020_1xAAA"
+		(property "Footprint" "Mylibrary:Batt terminal pads"
 			(at 66.04 61.976 90)
 			(hide yes)
